File: pcb-guide.kicad_sch (KiCad schematic)
At the start: 14 parts, among them SW1 SW_Push, U1 ATmega32U4-A, Y1 16MHz

Commit message: aaa
Parts:
- added D1, D2, D3, D4: D_Small, Diode_SMD:D_SOD-123, symbol Device:D_Small
- added F1: 500mA, Fuse:Fuse_1206_3216Metric, symbol Device:Polyfuse_Small
- added MX1, MX2, MX3, MX4: MX-NoLED, symbol MX_Alps_Hybrid:MX-NoLED
- added USB1: Molex-0548190589, symbol random-keyboard-parts:Molex-0548190589
- C1, C2: footprint (none) -> Capacitor_SMD:C_0805_2012Metric
- C3: renamed from 0.1uF; value C_Small -> 0.1uF; footprint (none) -> Capacitor_SMD:C_0805_2012Metric
- C4: renamed from 0.1uF1; value C_Small -> 0.1uF; footprint (none) -> Capacitor_SMD:C_0805_2012Metric
- C5: renamed from 0.1uF2; value C_Small -> 0.1uF; footprint (none) -> Capacitor_SMD:C_0805_2012Metric
- C6: renamed from 10uF; value C_Small -> 10uF; footprint (none) -> Capacitor_SMD:C_0805_2012Metric
- C7: renamed from 1uF; value C_Small -> 1uF; footprint (none) -> Capacitor_SMD:C_0805_2012Metric
- R1, R2: footprint (none) -> Resistor_SMD:R_0805_2012Metric
- R3: value 22 -> 10k; footprint (none) -> Resistor_SMD:R_0805_2012Metric
- R4: renamed from 10k; value R_Small -> 10k; footprint (none) -> Resistor_SMD:R_0805_2012Metric
Connections:
- net GND: now also USB1.1 (GND)
- net D+: now reaches R1.1
- net D+: now also USB1.3 (D+)
- net D-: now reaches R2.1
- net D-: now also USB1.4 (D-)
- new net: D3.2 (A), MX3.2 (ROW)
- new net: D2.2 (A), MX2.2 (ROW)
- new net: F1.1, USB1.5 (VBUS)
- new net: D3.1 (K), D4.1 (K)
- new net: D1.2 (A), MX1.2 (ROW)
- new net: MX1.1 (COL), MX4.1 (COL)
- new net: D4.2 (A), MX4.2 (ROW)
- new net VCC: F1.2
